Commit message: Descripiton clean up

File: src/description/urdf/Arm Full Assembly.urdf (robot description, URDF)
Before this commit: robot Arm Full Assembly, 4 links, 3 joints
Links:
- link base_link: geometry collision mesh filename=src/description/meshes/base_link.STL; visual mesh filename=src/description/meshes/base_link.STL
- link hand link: geometry collision mesh filename=src/description/meshes/hand_link.STL; visual mesh filename=src/description/meshes/hand_link.STL
- link link 1: geometry collision mesh filename=src/description/meshes/link_1.STL; visual mesh filename=src/description/meshes/link_1.STL
- link link 2: geometry collision mesh filename=src/description/meshes/link_2.STL; visual mesh filename=src/description/meshes/link_2.STL

Commit message: changed the urdf file

File: src/description/urdf/Arm Full Assembly.urdf (robot description, URDF)
Before this commit: robot arm_full_assembly, 4 links, 3 joints
Links:
- link base_link: geometry collision mesh filename=description/meshes/base_link.STL; visual mesh filename=description/meshes/base_link.STL
- link hand link: geometry collision mesh filename=description/meshes/hand_link.STL; visual mesh filename=description/meshes/hand_link.STL
- link link 1: geometry collision mesh filename=description/meshes/link_1.STL; visual mesh filename=description/meshes/link_1.STL
- link link 2: geometry collision mesh filename=description/meshes/link_2.STL; visual mesh filename=description/meshes/link_2.STL

Commit message: urdf file fixed

File: src/description/urdf/Arm Full Assembly.urdf (robot description, URDF)
Before this commit: robot arm_full_assembly, 4 links, 3 joints
Links:
- link base_link: geometry collision mesh filename=package://description/meshes/base_link.STL; visual mesh filename=package://description/meshes/base_link.STL
- link hand link: geometry collision mesh filename=package://description/meshes/hand_link.STL; visual mesh filename=package://description/meshes/hand_link.STL
- link link 1: geometry collision mesh filename=package://description/meshes/link_1.STL; visual mesh filename=package://description/meshes/link_1.STL
- link link 2: geometry collision mesh filename=package://description/meshes/link_2.STL; visual mesh filename=package://description/meshes/link_2.STL
