Commit message: Something works lol

File: src/description/urdf/new_arm_assembly.urdf (robot description, URDF)
Before this commit: robot Arm_Assembly, 2 links, 1 joints
Joints:
- removed joint base_to_link
- added joint shoulder: type revolute, parent base_link, child link_1, origin xyz=0 0 0.03935 rpy=-1.5708 0 -1.5708, axis 0 1 0, limit lower=-1.57 upper=1.57 effort=10 velocity=1

Commit message: second link possibly working

File: src/description/urdf/new_arm_assembly.urdf (robot description, URDF)
Before this commit: robot Arm_Assembly, 2 links, 1 joints
Links:
- added link link_2; visual mesh filename=package://description/meshes/link_2.STL
Joints:
- added joint elbow: type revolute, parent link_1, child link_2, origin xyz=-0.34315 -0.07335 -0.037841 rpy=0 0 -3.1416, axis 1 0 0, limit lower=-1.57 upper=1.57 effort=10 velocity=1

Commit message: Push

File: src/description/urdf/new_arm_assembly.urdf (robot description, URDF)
Before this commit: robot Arm_Assembly, 3 links, 2 joints
Links:
- added link hand_link; visual mesh filename=package://description/meshes/hand_link.STL
Joints:
- joint elbow: axis 1 0 0 -> 0 0 1

Commit message: URDF 3D model working Note: URDF file needs update

File: src/description/urdf/new_arm_assembly.urdf (robot description, URDF)
Before this commit: robot Arm_Assembly, 4 links, 2 joints
Links:
- removed link hand_link

Commit message: New URDF

File: src/description/urdf/new_arm_assembly.urdf (robot description, URDF)
Before this commit: robot Arm_Assembly, 3 links, 2 joints
Links:
- added link base_joint, mass 1.4774; collision mesh filename=package://description/meshes/base_joint.STL; visual mesh filename=package://description/meshes/base_joint.STL
- added link link_3, mass 2.0738; collision mesh filename=package://description/meshes/link_3.STL; visual mesh filename=package://description/meshes/link_3.STL
- added link link_4, mass 1.5647; collision mesh filename=package://description/meshes/link_4.STL; visual mesh filename=package://description/meshes/link_4.STL
- added link link_5, mass 0.75097; collision mesh filename=package://description/meshes/link_5.STL; visual mesh filename=package://description/meshes/link_5.STL
- link base_link: mass None -> 0.69252; geometry collision mesh filename=package://description/meshes/base_link.STL; visual mesh filename=package://description/meshes/base_link.STL
- link link_1: mass None -> 3.4436; geometry collision mesh filename=package://description/meshes/link_1.STL; visual mesh filename=package://description/meshes/link_1.STL
- link link_2: mass None -> 1.5154; geometry collision mesh filename=package://description/meshes/link_2.STL; visual mesh filename=package://description/meshes/link_2.STL
Joints:
- removed joint elbow
- removed joint shoulder
- added joint Elbow Roll: type revolute, parent link_2, child link_3, origin xyz=-0.031996 -0.11212 -0.10012 rpy=0 0.28935 -0.22538, axis 0 1 0, limit lower=-3.14159 upper=3.14159 effort=0 velocity=0
- added joint Elbow Yaw: type revolute, parent link_1, child link_2, origin xyz=-0.32046 -0.18979 0.054866 rpy=-0.066431 -0.28183 -2.9068, axis 0.22347 0.97471 0, limit lower=-2.79253 upper=1.97222 effort=0 velocity=0
- added joint Shoulder Roll: type continuous, parent base_link, child base_joint, origin xyz=0 0 0 rpy=0.74076 -1.5708 0, axis 1 0 0
- added joint Shoulder Yaw: type revolute, parent base_joint, child link_1, origin xyz=0.03935 0 0 rpy=0 -0.74076 1.5708, axis 0 -1 0, limit lower=-1.0472 upper=3.66519 effort=0 velocity=0
- added joint Wrist Pitch: type revolute, parent link_3, child link_4, origin xyz=0.24203 -0.10445 0.026121 rpy=2.6277 0.12902 0.0099744, axis 0.0098913 -0.87017 -0.49266, limit lower=-2.75762 upper=2.67035 effort=0 velocity=0
- added joint Wrist Roll: type continuous, parent link_4, child link_5, origin xyz=0.10059 -0.10682 -0.32961 rpy=-2.5237 -0.79049 1.6048, axis -0.96217 -0.17349 -0.21007, limit lower=0 upper=0 effort=0 velocity=0

Commit message: just a save

File: src/description/urdf/new_arm_assembly.urdf (robot description, URDF)
Before this commit: robot Arm Full Assembly V3, 7 links, 6 joints
Joints:
- joint Elbow Yaw: axis 0.22347 0.97471 0 -> 0 0 1

Commit message: IT WORKSSSS URDF

File: src/description/urdf/new_arm_assembly.urdf (robot description, URDF)
Before this commit: robot Arm Full Assembly V3, 7 links, 6 joints
Links:
- link base_joint: mass 1.4774 -> 1.47738507112296
- link base_link: mass 0.69252 -> 0.692524123906466
- link link_1: mass 3.4436 -> 3.44363478464573
- link link_2: mass 1.5154 -> 1.5153745049325
- link link_3: mass 2.0738 -> 2.07375542707273
- link link_4: mass 1.5647 -> 1.56472201375409
- link link_5: mass 0.75097 -> 0.750967399035288
Joints:
- removed joint Elbow Yaw
- removed joint Shoulder Yaw
- added joint Elbow Pitch: type revolute, parent link_1, child link_2, origin xyz=0.0428412022704851 -0.000700000000055892 -0.34315000105285 rpy=0 0 -3.14159265358978, axis 1 0 0, limit lower=-2.7925 upper=1.9722 effort=0 velocity=0
- added joint Shoulder Pitch: type revolute, parent base_joint, child link_1, origin xyz=0.112 0 0 rpy=0 0.830034063284424 1.57079632679488, axis -1 0 0, limit lower=-1.0472 upper=3.6652 effort=0 velocity=0
- joint Elbow Roll: axis 0 1 0 -> 1 0 0; limit lower=-3.14159 upper=3.14159 effort=0 velocity=0 -> lower=-3.1416 upper=3.1416 effort=0 velocity=0; origin xyz=-0.031996 -0.11212 -0.10012 rpy=0 0.28935 -0.22538 -> xyz=0.09 0 0 rpy=1.5707963267949 1.5707963267949 0
- joint Shoulder Roll: origin xyz=0 0 0 rpy=0.74076 -1.5708 0 -> xyz=0 0 0 rpy=0.740762263510472 -1.5707963267949 0
- joint Wrist Pitch: axis 0.0098913 -0.87017 -0.49266 -> -1 0 0; limit lower=-2.75762 upper=2.67035 effort=0 velocity=0 -> lower=-2.7576 upper=2.6704 effort=0 velocity=0; origin xyz=0.24203 -0.10445 0.026121 rpy=2.6277 0.12902 0.0099744 -> xyz=0.25884999894715 -0.00284120227048547 0.000299999999948689 rpy=-1.57079632679492 0 1.5707963267949
- joint Wrist Roll: axis -0.96217 -0.17349 -0.21007 -> 1 0 0; origin xyz=0.10059 -0.10682 -0.32961 rpy=-2.5237 -0.79049 1.6048 -> xyz=0.09 0.00300000000000089 0.002 rpy=1.57079632679489 1.5707963267949 0
