Commit message: URDF updated with new eef link

File: src/description/urdf/SPEAR_Arm.urdf (robot description, URDF)
Before this commit: robot SPEAR_Arm, 7 links, 6 joints
Links:
- added link EEF; collision box size=0.02 0.02 0.02; visual box size=0.02 0.02 0.02
Joints:
- added joint EEF_Joint: type fixed, parent link_5, child EEF, origin xyz=0.01 0 0 rpy=1.57079632679489 1.5707963267949 0

Commit message: Arm axis adjusted

File: src/description/urdf/SPEAR_Arm.urdf (robot description, URDF)
Before this commit: robot SPEAR_Arm, 8 links, 7 joints
Joints:
- joint Elbow Pitch: axis 1 0 0 -> 0 1 0; origin xyz=0.0428412022704851 -0.000700000000055892 -0.34315000105285 rpy=0 0 -3.14159265358978 -> xyz=-0.34315 -0.0428412022704851 0.000700000000055892 rpy=0 0 0
- joint Elbow Roll: origin xyz=0.09 0 0 rpy=1.5707963267949 1.5707963267949 0 -> xyz=0 0.09 0 rpy=0 0 0
- joint Shoulder Pitch: axis -1 0 0 -> 0 1 0; origin xyz=0.112 0 0 rpy=0 0.830034063284424 1.57079632679488 -> xyz=0 0 0.112 rpy=0 0 0
- joint Shoulder Roll: axis 1 0 0 -> 0 0 1; origin xyz=0 0 0 rpy=0.740762263510472 -1.5707963267949 0 -> xyz=0 0 0 rpy=0 0 0
- joint Wrist Pitch: axis -1 0 0 -> 0 1 0; origin xyz=0.25884999894715 -0.00284120227048547 0.000299999999948689 rpy=-1.57079632679492 0 1.5707963267949 -> xyz=-0.25884999894715 -0.00284120227048547 -0.000299999999948689 rpy=0 0 0
- joint Wrist Roll: origin xyz=0.09 0.00300000000000089 -0.25 rpy=1.57079632679489 1.5707963267949 0 -> xyz=-0.25 0.09 0.00300000000000089 rpy=0 0 0

Commit message: Mesh and Links complete

File: src/description/urdf/SPEAR_Arm.urdf (robot description, URDF)
Before this commit: robot SPEAR_Arm, 8 links, 7 joints
Joints:
- joint EEF_Joint: origin xyz=0.01 0 0 rpy=1.57079632679489 1.5707963267949 0 -> xyz=-0.01 0 0 rpy=0 0 0

Commit message: update

File: src/description/urdf/SPEAR_Arm.urdf (robot description, URDF)
Before this commit: robot SPEAR_Arm, 8 links, 7 joints
Links:
- link link_1: geometry collision box size=0.14 0.08 0.1; visual mesh filename=package://description/meshes/link_1.STL
- link link_2: geometry collision box size=0.1 0.1 0.08; visual mesh filename=package://description/meshes/link_2.STL

Commit message: urdf collision updated

File: src/description/urdf/SPEAR_Arm.urdf (robot description, URDF)
Before this commit: robot SPEAR_Arm, 8 links, 7 joints
Links:
- link link_1: geometry collision box size=0.14 0.08 0.055; visual mesh filename=package://description/meshes/link_1.STL
- link link_4: geometry collision box size=0.16 0.082 0.08; visual mesh filename=package://description/meshes/link_4.STL
