Commit message: Joy inpust being taken

File: src /description/urdf/SPEAR_Arm.urdf (robot description, URDF)
Before this commit: robot SPEAR_Arm, 7 links, 6 joints
Links:
- link base_joint: geometry collision mesh filename=package://description/meshes/joint_1_collsion.STL; visual mesh filename=package://description/meshes/base_joint.STL
- link base_link: geometry collision mesh filename=package://description/meshes/base_link_collision.STL; visual mesh filename=package://description/meshes/base_link.STL

Commit message: URDF working

File: src /description/urdf/SPEAR_Arm.urdf (robot description, URDF)
Before this commit: robot SPEAR_Arm, 7 links, 6 joints
Links:
- link base_joint: geometry collision box size=0.121 0.11 0.11; visual mesh filename=package://description/meshes/base_joint.STL
- link base_link: geometry collision box size=0.128 0.128 0.07; visual mesh filename=package://description/meshes/base_link.STL
- link link_1: geometry collision box size=0.1 0.08 0.14; visual mesh filename=package://description/meshes/link_1.STL
- link link_2: geometry collision box size=0.1 0.08 0.1; visual mesh filename=package://description/meshes/link_2.STL
- link link_3: geometry collision box size=0.21 0.08 0.084; visual mesh filename=package://description/meshes/link_3.STL
- link link_4: geometry collision box size=0.08 0.082 0.16; visual mesh filename=package://description/meshes/link_4.STL
- link link_5: geometry collision box size=0.16 0.08 0.14; visual mesh filename=package://description/meshes/link_5.STL
Joints:
- joint Wrist Roll: origin xyz=0.09 0.00300000000000089 0.002 rpy=1.57079632679489 1.5707963267949 0 -> xyz=0.09 0.00300000000000089 -0.25 rpy=1.57079632679489 1.5707963267949 0

Commit message: URDF EEF LINK ADDED

File: src /description/urdf/SPEAR_Arm.urdf (robot description, URDF)
Before this commit: robot SPEAR_Arm, 7 links, 6 joints
Links:
- added link eef_link; collision box size=0.01 0.01 0.01; visual box size=0.01 0.01 0.01
Joints:
- added joint eef_joint: type fixed, parent link_5, child eef_link, origin xyz=0.17 0 0 rpy=1.57079632679489 1.5707963267949 0
- joint Wrist Roll: origin xyz=0.09 0.00300000000000089 -0.25 rpy=1.57079632679489 1.5707963267949 0 -> xyz=0.09 0.00300000000000089 -0.12 rpy=1.57079632679489 1.5707963267949 0

Commit message: ARm working with controls kindda

File: src /description/urdf/SPEAR_Arm.urdf (robot description, URDF)
Before this commit: robot SPEAR_Arm, 8 links, 7 joints
Links:
- removed link eef_link
Joints:
- removed joint eef_joint
- joint Wrist Roll: origin xyz=0.09 0.00300000000000089 -0.12 rpy=1.57079632679489 1.5707963267949 0 -> xyz=0.09 0.00300000000000089 -0.25 rpy=1.57079632679489 1.5707963267949 0
